File: DeWinCNC.sch (KiCad schematic (older format))
At the start: 87 parts, among them J1 Digital, J10 Vcc, J11 S3, J12 Aux-1a, J13 S4, J14 X-axis, J15 Y-axis, J16 Z-axis, J18 A-axis, J19 X-, J2 Aux-4, J20 X+, J21 Y-, J22 Y+, J23 Z-, J24 Z+, J25 B-axis, J261 RLA2, J262 RLA3, J27 T1 T2 T3, J28 RLA1, J29 I2C, J3 S1, J30 RLA4, J31 0V / 5V, J32 0V / 5V, J33 0V / 5V, J34 0V / 5V, J35 0V / 5V, J36 PWM, J37 1-Wire, J38 IDC for DB37, J39 D7, J4 Vcc, J40 Limits, J41 Limit, J42 Limit, J43 Limit, J44 Limit, J45 Limit, J46 Limit, J47 1-Wire, J5 5v,PS_ON,Vcc, J6 Aux-1b, J7 S2, J8 Aux-2, J9 Aux-3, P10 CONN_01X01, P11 CONN_01X01, SW1 RESET, U1 S102S01, U2 S102S01, U3 S102S01, U4 S102S01, U5 LM7812_TO220

Commit message: Update ESP pinout, round edges more.
Parts:
- added J50: 3.3v, symbol Connector:Conn_01x01_Male
- added J51: Serial0, symbol Connector_Generic:Conn_01x05
- added J52: DB15_Joystick, symbol Connector:DB15_Female_MountingHoles
- added JP48: D56,D57,D62?, symbol Jumper:SolderJumper_2_Bridged
- added JP49: Laser/Spindle, symbol Jumper:SolderJumper_2_Bridged
- added U1001: ESP-01v090, Connector_PinSocket_2.54mm:PinSocket_2x04_P2.54mm_Vertical, symbol ESP8266:ESP-01v090
Connections:
- net +5V: now also J51.1 (Pin_1), J52.1
- net D0(Rx0): now also J51.4 (Pin_4), U1001.8 (GPIO1)
- net D1(Tx0): now also J51.3 (Pin_3), U1001.4 (GPIO3)
- net D22: now also JP48.2 (B); no longer J37.2 (Pin_2), J47.2 (Pin_2), R10.2
- net D44: now also JP49.2 (B); no longer J36.1 (Pin_1)
- net D56(A2): now also J52.7
- net D57(A3): now also J52.3
- net D58(A4): now also J52.6
- net D62(A8): now also J52.2
- net GND: now also J51.2 (Pin_2), J52.0 (PAD), J52.4, J52.5, U1001.1 (GND)
- net 3.3v: now reaches JM5.4 (Pin_4)
- net 3.3v: now also J50.1 (Pin_1), J51.5 (Pin_5), U1001.5 (VCC), U1001.7 (CH_PD)
- new net: J37.2 (Pin_2), J47.2 (Pin_2), JP48.1 (A), R10.2
- new net: J36.1 (Pin_1), JP49.1 (A)
- no-connect marks 20 -> 28
Other:
- moved on the sheet: R10
